File: regulators.sch (KiCad schematic (older format))
At the start: 4 parts, among them J6 Power_output, U2 lm2596_blue_board

Commit message: fixing wrong diode symbol for simulation only
Changed lines of the file:
@@
 AR Path="/615A8E56/6159A2FA" Ref="F8"  Part="1"
 AR Path="/615ABAD5/6159A2FA" Ref="F9"  Part="1"
-F 0 "F6" V 5053 3600 50  0000 C CNN
+F 0 "F9" V 5053 3600 50  0000 C CNN
 F 1 "Fuse" V 5144 3600 50  0000 C CNN
 F 2 "Fuse:Fuse_Littelfuse_372_D8.50mm" V 5180 3600 50  0001 C CNN
@@
 AR Path="/615A8E56/6159A911" Ref="J9"  Part="1"
 AR Path="/615ABAD5/6159A911" Ref="J10"  Part="1"
-F 0 "J7" H 6180 3492 50  0000 L CNN
+F 0 "J10" H 6180 3492 50  0000 L CNN
 F 1 "Power_output" H 6180 3401 50  0000 L CNN
 F 2 "Connector_Phoenix_MC:PhoenixContact_MC_1,5_2-G-3.81_1x02_P3.81mm_Horizontal" H 6100 3500 50  0001 C CNN
@@
 AR Path="/615A8E56/6159B24E" Ref="#PWR028"  Part="1"
 AR Path="/615ABAD5/6159B24E" Ref="#PWR031"  Part="1"
-F 0 "#PWR022" H 5900 3250 50  0001 C CNN
+F 0 "#PWR031" H 5900 3250 50  0001 C CNN
 F 1 "GND" V 5905 3372 50  0000 R CNN
 F 2 "" H 5900 3500 50  0001 C CNN
@@
 AR Path="/615A8E56/615A0D04" Ref="JP6"  Part="1"
 AR Path="/615ABAD5/615A0D04" Ref="JP7"  Part="1"
-F 0 "JP4" V 3096 3687 50  0000 L CNN
+F 0 "JP7" V 3096 3687 50  0000 L CNN
 F 1 "Jumper_3_Open" V 3005 3687 50  0000 L CNN
 F 2 "Connector_PinHeader_2.54mm:PinHeader_1x03_P2.54mm_Vertical" H 3050 3600 50  0001 C CNN
@@
 AR Path="/615A8E56/615A1E14" Ref="U5"  Part="1"
 AR Path="/615ABAD5/615A1E14" Ref="U6"  Part="1"
-F 0 "U3" H 4175 4065 50  0000 C CNN
+F 0 "U6" H 4175 4065 50  0000 C CNN
 F 1 "lm2596_blue_board" H 4175 3974 50  0000 C CNN
 F 2 "kiwi_power:lm2596_blue_board" H 4200 3700 50  0001 C CNN
@@
 AR Path="/615A8E56/615A247F" Ref="#PWR027"  Part="1"
 AR Path="/615ABAD5/615A247F" Ref="#PWR030"  Part="1"
-F 0 "#PWR021" H 4700 3650 50  0001 C CNN
+F 0 "#PWR030" H 4700 3650 50  0001 C CNN
 F 1 "GND" V 4705 3772 50  0000 R CNN
 F 2 "" H 4700 3900 50  0001 C CNN
@@
 AR Path="/615A8E56/615A29A4" Ref="#PWR026"  Part="1"
 AR Path="/615ABAD5/615A29A4" Ref="#PWR029"  Part="1"
-F 0 "#PWR020" H 3650 3650 50  0001 C CNN
+F 0 "#PWR029" H 3650 3650 50  0001 C CNN
 F 1 "GND" V 3655 3772 50  0000 R CNN
 F 2 "" H 3650 3900 50  0001 C CNN
@@
 AR Path="/615A8E56/615BB707" Ref="#FLG0106"  Part="1"
 AR Path="/615ABAD5/615BB707" Ref="#FLG0107"  Part="1"
-F 0 "#FLG0104" H 3400 3675 50  0001 C CNN
+F 0 "#FLG0107" H 3400 3675 50  0001 C CNN
 F 1 "PWR_FLAG" H 3400 3773 50  0000 C CNN
 F 2 "" H 3400 3600 50  0001 C CNN

Commit message: version 2
Changed lines of the file:
@@
 $Descr A4 11693 8268
 encoding utf-8
-Sheet 6 9
+Sheet 5 9
 Title ""
 Date ""
@@
 AR Path="/615A8E56/6159A2FA" Ref="F8"  Part="1"
 AR Path="/615ABAD5/6159A2FA" Ref="F9"  Part="1"
-F 0 "F9" V 5053 3600 50  0000 C CNN
+F 0 "F5" V 5053 3600 50  0000 C CNN
 F 1 "Fuse" V 5144 3600 50  0000 C CNN
 F 2 "Fuse:Fuse_Littelfuse_372_D8.50mm" V 5180 3600 50  0001 C CNN
@@
 AR Path="/615A8E56/6159A911" Ref="J9"  Part="1"
 AR Path="/615ABAD5/6159A911" Ref="J10"  Part="1"
-F 0 "J10" H 6180 3492 50  0000 L CNN
+F 0 "J6" H 6180 3492 50  0000 L CNN
 F 1 "Power_output" H 6180 3401 50  0000 L CNN
 F 2 "Connector_Phoenix_MC:PhoenixContact_MC_1,5_2-G-3.81_1x02_P3.81mm_Horizontal" H 6100 3500 50  0001 C CNN
@@
 AR Path="/615A8E56/615A0D04" Ref="JP6"  Part="1"
 AR Path="/615ABAD5/615A0D04" Ref="JP7"  Part="1"
-F 0 "JP7" V 3096 3687 50  0000 L CNN
+F 0 "JP3" V 3096 3687 50  0000 L CNN
 F 1 "Jumper_3_Open" V 3005 3687 50  0000 L CNN
 F 2 "Connector_PinHeader_2.54mm:PinHeader_1x03_P2.54mm_Vertical" H 3050 3600 50  0001 C CNN
@@
 AR Path="/615A8E56/615A1E14" Ref="U5"  Part="1"
 AR Path="/615ABAD5/615A1E14" Ref="U6"  Part="1"
-F 0 "U6" H 4175 4065 50  0000 C CNN
+F 0 "U2" H 4175 4065 50  0000 C CNN
 F 1 "lm2596_blue_board" H 4175 3974 50  0000 C CNN
 F 2 "kiwi_power:lm2596_blue_board" H 4200 3700 50  0001 C CNN
